File: PCB/pcb_transitoire/pcb_transitoire.kicad_sch (KiCad schematic)
At the start: 28 parts, among them J1 OpticalSensorIn, J10 Shutter_Motor, J11 Arduino_GPIO_Shutter, J12 GRATING_MOTOR, J13 SLIT1_MOTOR, J14 SLIT2_MOTOR, J15 SLIT3_MOTOR, J16 ARDUINO SHIELD_Z, J17 ARDUINO SHIELD_A, J18 ARDUINO SHIELD_Y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

Commit message: Ajout des dernières ressources manquantes
Other:
- title: PCB de connection pour carte Arduino -> PCB de connexion pour carte Arduino
Changed lines of the file:
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@@
 	(paper "A4")
 	(title_block
-		(title "PCB de connection pour carte Arduino")
+		(title "PCB de connexion pour carte Arduino")
 		(date "19/06/2025")
 		(rev "1.0")
